File: Hardware/SparrowAprs.sch (EAGLE design)
At the start: 87 parts, among them IC1 STM32F40X_LQFP64, IC2 NEO-M8, IC3 TPS62142RGTT, IC4 BME280, J1 USB_MINI-B_SMT, J3 DF13-6P-1.25H, J4 FSK_RUARK2_SMA_0732511150, J5 FSK_RUARK2_SMA_0732511150, SW1 TAC_SWITCH, U3 DRA818V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

Commit message: New hardware rev
Parts:
- removed C37, C38: 10uF, resistor:C-EUC0805
- removed R28: 0R, resistor:R-US_R0805
- added U$5: HEADER_6_JSTGH, HappyMedium:HEADER_6_JSTGH
- J3: value DF13-6P-1.25H -> (none); device con-hirose-df13:DF13-6P-1.25H -> SparkFun-Connectors:CONN_02
- R2: value 100R -> 1M
- SW1: value TAC_SWITCH -> 1825027-8; device HappyMedium:TAC_SWITCH -> button:1825027-8
Connections:
- removed net 3V3_ISO: C29.1, C30.1, IC3.FSW, IC3.VOS, L2.1, R28.1
- removed net N$6: IC1.BOOT0, R5.2
- new net BOOT0: IC1.BOOT0, J3.1, R5.2
- net +3V3: now also C29.1, C30.1, IC3.FSW, IC3.VOS, L2.1, U$5.5; no longer C37.1, C38.1, R28.2
- net EXT1: now also U$5.4; no longer J3.3
- net EXT2: now also U$5.3; no longer J3.4
- net EXT3: now also U$5.2; no longer J3.5
- net EXT4: now also U$5.1; no longer J3.6
- net GND: now also IC1.PB2, SW1.2, SW1.3, SW1.4, U$5.6; no longer C37.2, C38.2, J3.1, SW1.P$2
- net MCU_BUTTON: now also SW1.1; no longer SW1.P$1
- net N$11: no longer R2.2
- net N$14: now also R2.2
Other:
- note added: "PB2 is BOOT1. Keep low"
- note removed: "PSU Isolation"
- moved on the sheet: C1, R2, R3, R5
