File: Hardware/SparrowAprs.brd (EAGLE design)
At the start: 66.7 x 54.4 mm, 87 parts, among them IC1 STM32F40X_LQFP64, IC2 NEO-M8, IC3 TPS62142RGTT, IC4 BME280, J1 USB_MINI-B_SMT, J3 DF13-6P-1.25H, J4 FSK_RUARK2_SMA_0732511150, J5 FSK_RUARK2_SMA_0732511150, SW1 TAC_SWITCH, U3 DRA818V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

Commit message: New hardware rev
Parts:
- removed C37, C38: 10uF, resistor:C0805
- removed R28: 0R, resistor:R0805
- added U$5: HEADER_6_JSTGH, HappyMedium:BM06B-GHS-TBT(LF)(SN)(N)
- J3: value DF13-6P-1.25H -> (none); device con-hirose-df13:DF13A-6P-1.25H -> SparkFun-Connectors:1X02
- R2: value 100R -> 1M
- SW1: value TAC_SWITCH -> 1825027-8; device HappyMedium:EVQP7B -> button:SW2_1825027-C
- moved J3 35.5 mm to (10.9, 31.4), turned to 270 degrees
- moved U$1 27.1 mm to (50.6, 50.3), flipped to the top, turned to 270 degrees
- moved R2 8.45 mm to (26.2, 26.0)
- moved R9 7.81 mm to (58.4, 46.9)
- moved R27 2.93 mm to (42.5, 46.8)
- moved J2 2.92 mm to (3.62, 13.6)
- moved R26 2.87 mm to (38.5, 46.8)
- moved R3 2.16 mm to (34.7, 26.0)
- moved C1 2.03 mm to (32.0, 26.0)
- moved C24 1.91 mm to (29.0, 26.0)
- moved D5 1.47 mm to (10.9, 23.2), turned to 90 degrees
- moved SW1 1.40 mm to (2.79, 26.3), turned to 270 degrees
- moved U$7 0.51 mm to (3.81, 51.1)
- moved U$9 0.51 mm to (62.9, 51.1)
- moved R11 0.44 mm to (21.9, 26.0)
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Connections:
- removed net 3V3_ISO: C29.1, C30.1, IC3.14, IC3.7, L2.1, R28.1
- removed net N$6: IC1.60, R5.2
- new net BOOT0: IC1.60, J3.1, R5.2
- net +3V3: now also C29.1, C30.1, IC3.14, IC3.7, J3.2, L2.1, U$5.5; no longer C37.1, C38.1, J3.P$2, R28.2
- net EXT1: now also U$5.4; no longer J3.P$3
- net EXT2: now also U$5.3; no longer J3.P$4
- net EXT3: now also U$5.2; no longer J3.P$5
- net EXT4: now also U$5.1; no longer J3.P$6
- net GND: now also IC1.28, SW1.3, SW1.4, U$5.6; no longer C37.2, C38.2, J3.P$1
- net N$11: no longer R2.2
- net N$14: now also R2.2
Routing:
- net DEBUG_USART_TX: track 11.7 -> 46.7 mm, vias 1 -> 2
- net !NRST: track 14.1 -> 47.0 mm, vias 1 -> 2
- net SWD_SWDIO: track 8.11 -> 36.5 mm, vias 1 -> 2
- net SWD_SWCLK: track 12.6 -> 33.0 mm, vias 1 -> 2
- net BOOT0: track 0.00 -> 13.4 mm
- net 3V3_ISO: track 9.82 -> 0.00 mm, vias 8 -> 0
- net N$10: track 11.7 -> 3.92 mm
- net +3V3: track 50.0 -> 57.7 mm, vias 49 -> 52
- net NEO_PPS: track 36.9 -> 43.4 mm
- net N$14: track 24.4 -> 30.0 mm
- net N$18: track 10.0 -> 5.97 mm
- net EXT3: track 35.1 -> 31.7 mm
- net EXT4: track 37.6 -> 34.3 mm
- net EXT2: track 21.4 -> 18.3 mm
- net EXT1: track 19.4 -> 16.4 mm
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- added copper zone on layer 1, net +3V3
- removed copper zone on layer 16, net +3V3
- removed copper zone on layer 1, net 3V3_ISO
- removed copper zone on layer 16, net 3V3_ISO
Other:
- board size 66.7 x 54.4 mm -> 66.7 x 54.9 mm
- board text added: "PPS"
- board text removed: "GPS PPS"

Commit message: Updated hardware
Parts:
- removed U$1: HEADER_6, HappyMedium:6X2_SMT
- added JMP1: (no value), SparkFun-Connectors:1X02
- J3: value (none) -> HEADER_6; device SparkFun-Connectors:1X02 -> HappyMedium:6X2_SMT
- moved J3 44.0 mm to (50.6, 50.3)
- moved C36 2.50 mm to (52.8, 26.6), turned to 270 degrees
- renumbered U$5 to J6, U3 to IC5
Connections:
- net !NRST: now also J3.3; no longer U$1.3
- net +3V3: now also J3.6, JMP1.2; no longer J3.2, U$1.6
- net BOOT0: now also JMP1.1; no longer J3.1
- net DEBUG_USART_TX: now also J3.4; no longer U$1.4
- net GND: now also J3.1; no longer U$1.1
- net SWD_SWCLK: now also J3.2; no longer U$1.2
- net SWD_SWDIO: now also J3.5; no longer U$1.5
Routing:
- net NEO_PPS: track 43.4 -> 44.1 mm
- net SWD_SWDIO: track 36.5 -> 36.0 mm
Other:
- board text removed: "T"
